Commit message: cyphal injected

File: config/diffbot.ros2_control.xacro (robot description, xacro)
@@ -1,5 +1,5 @@
 <?xml version="1.0"?>
 <robot xmlns:xacro="http://www.ros.org/wiki/xacro">
-  <xacro:macro name="diffbot_ros2_control" params="name prefix use_mock_hardware">
+  <xacro:macro name="diffbot_ros2_control" params="name prefix dont_use_mock_hardware">
     <ros2_control name="${name}" type="system">
       <xacro:unless value="${use_mock_hardware}">

Commit message: new urdf

File: config/diffbot.ros2_control.xacro (robot description, xacro)
@@ -1,25 +1,26 @@
 <?xml version="1.0"?>
 <robot xmlns:xacro="http://www.ros.org/wiki/xacro">
-  <xacro:macro name="diffbot_ros2_control" params="name prefix dont_use_mock_hardware">
+  <xacro:macro name="diffbot_ros2_control" params="name">
+    <!-- <xacro:property name="initial_positions" value="${xacro.load_yaml(initial_positions_file)['initial_positions']}"/> -->
     <ros2_control name="${name}" type="system">
-      <xacro:unless value="${use_mock_hardware}">
+      <!-- <xacro:unless value="${use_mock_hardware}"> -->
         <hardware>
-          <plugin>ros2_control_demo_example_2/DiffBotSystemHardware</plugin>
-          <param name="example_param_hw_start_duration_sec">0</param>
-          <param name="example_param_hw_stop_duration_sec">3.0</param>
+          <plugin>diffbot/DiffBotSystemHardware</plugin>
+          <!-- <param name="example_param_hw_start_duration_sec">0</param>
+          <param name="example_param_hw_stop_duration_sec">3.0</param> -->
         </hardware>
-      </xacro:unless>
-      <xacro:if value="${use_mock_hardware}">
+      <!-- </xacro:unless> -->
+      <!-- <xacro:if value="${use_mock_hardware}">
         <hardware>
           <plugin>mock_components/GenericSystem</plugin>
           <param name="calculate_dynamics">true</param>
         </hardware>
-      </xacro:if>
-      <joint name="${prefix}left_wheel_joint">
+      </xacro:if> -->
+      <joint name="left_wheel_joint">
         <command_interface name="velocity"/>
         <state_interface name="position"/>
         <state_interface name="velocity"/>
       </joint>
-      <joint name="${prefix}right_wheel_joint">
+      <joint name="right_wheel_joint">
         <command_interface name="velocity"/>
         <state_interface name="position"/>

File: config/diffbot.urdf.xacro (robot description, xacro)
@@ -1,14 +1,10 @@
 <?xml version="1.0"?>
 <!-- Basic differential drive mobile base -->
-<robot xmlns:xacro="http://www.ros.org/wiki/xacro" name="diffdrive_robot">
+<robot xmlns:xacro="http://www.ros.org/wiki/xacro" name="diffbot">
   <xacro:arg name="prefix" default="" />
-  <xacro:arg name="use_mock_hardware" default="false" />
   <xacro:include filename="$(find diffbot)/config/diffbot_description.urdf.xacro" />
-  <!-- Import Rviz colors -->
   <xacro:include filename="$(find diffbot)/config/diffbot.materials.xacro" />
-  <!-- Import diffbot ros2_control description -->
   <xacro:include filename="$(find diffbot)/config/diffbot.ros2_control.xacro" />
-  <xacro:diffbot prefix="$(arg prefix)" />
-  <xacro:diffbot_ros2_control
-    name="DiffBot" prefix="$(arg prefix)" use_mock_hardware="$(arg use_mock_hardware)"/>
+  <xacro:diffbot_ros2_control name="DiffBot" />
+  <!-- initial_positions_file="$(arg initial_positions_file)"/> -->
 </robot>

File: config/diffbot_description.urdf.xacro (robot description, xacro)
@@ -1,5 +1,4 @@
 <?xml version="1.0"?>
 <robot xmlns:xacro="http://www.ros.org/wiki/xacro">
-  <xacro:macro name="diffbot" params="prefix">
   <!-- Constants for robot dimensions -->
   <xacro:property name="PI" value="3.1415926535897931"/>
@@ -15,5 +14,5 @@
   <xacro:property name="z_offset" value="-${base_height/2}" /> <!-- Space btw top of beam and the each joint -->
   <!-- Base Link -->
-  <link name="${prefix}base_link">
+  <link name="base_link">
     <collision>
       <origin xyz="0 0 0" rpy="0 0 0"/>
@@ -38,7 +37,7 @@
       </inertial>
     </link>
-    <joint name="${prefix}left_wheel_joint" type="continuous">
-      <parent link="${prefix}base_link"/>
-      <child link="${prefix}left_wheel"/>
+    <joint name="left_wheel_joint" type="continuous">
+      <parent link="base_link"/>
+      <child link="left_wheel"/>
       <origin xyz="0 -${base_width/2} ${z_offset}" rpy="0 0 0"/>
       <axis xyz="0 1 0"/>
@@ -47,5 +46,5 @@
     </joint>
     <!-- left wheel Link -->
-    <link name="${prefix}left_wheel">
+    <link name="left_wheel">
       <collision>
         <origin xyz="0 0 0" rpy="${PI/2} 0 0"/>
@@ -70,7 +69,7 @@
         </inertial>
       </link>
-    <joint name="${prefix}right_wheel_joint" type="continuous">
-      <parent link="${prefix}base_link"/>
-      <child link="${prefix}right_wheel"/>
+    <joint name="right_wheel_joint" type="continuous">
+      <parent link="base_link"/>
+      <child link="right_wheel"/>
       <origin xyz="0 ${base_width/2} ${z_offset}" rpy="0 0 0"/>
       <axis xyz="0 1 0"/>
@@ -79,5 +78,5 @@
     </joint>
     <!-- right wheel Link -->
-    <link name="${prefix}right_wheel">
+    <link name="right_wheel">
       <collision>
         <origin xyz="0 0 0" rpy="${PI/2} 0 0"/>
@@ -102,11 +101,11 @@
         </inertial>
       </link>
-    <joint name="${prefix}caster_frontal_wheel_joint" type="fixed">
-      <parent link="${prefix}base_link"/>
-      <child link="${prefix}caster_frontal_wheel"/>
+    <joint name="caster_frontal_wheel_joint" type="fixed">
+      <parent link="base_link"/>
+      <child link="caster_frontal_wheel"/>
       <origin xyz="${base_width/2 - caster_wheel_radius} 0 ${z_offset}" rpy="0 0 0"/>
     </joint>
     <!-- caster frontal wheel Link -->
-    <link name="${prefix}caster_frontal_wheel">
+    <link name="caster_frontal_wheel">
       <collision>
         <origin xyz="0 0 0" rpy="0 0 0"/>
@@ -131,11 +130,11 @@
         </inertial>
       </link>
-    <joint name="${prefix}caster_rear_wheel_joint" type="fixed">
-      <parent link="${prefix}base_link"/>
-      <child link="${prefix}caster_rear_wheel"/>
+    <joint name="caster_rear_wheel_joint" type="fixed">
+      <parent link="base_link"/>
+      <child link="caster_rear_wheel"/>
       <origin xyz="${-base_width/2 + caster_wheel_radius} 0 ${z_offset}" rpy="0 0 0"/>
     </joint>
     <!-- caster rear wheel Link -->
-    <link name="${prefix}caster_rear_wheel">
+    <link name="caster_rear_wheel">
       <collision>
         <origin xyz="0 0 0" rpy="0 0 0"/>
@@ -160,4 +159,3 @@
         </inertial>
       </link>
-  </xacro:macro>
 </robot>

Commit message: stable

File: config/diffbot.ros2_control.xacro (robot description, xacro)
@@ -7,5 +7,5 @@
         <hardware>
           <plugin>diffbot/DiffBotSystemHardware</plugin>
-          <!-- <param name="example_param_hw_start_duration_sec">0</param>
+          <!-- <param name="zlp">0</param>
           <param name="example_param_hw_stop_duration_sec">3.0</param> -->
         </hardware>

File: config/diffbot_description.urdf.xacro (robot description, xacro)
@@ -28,5 +28,5 @@
       <material name="orange"/>
     </visual>
-    <inertial>
+    <!-- <inertial>
       <origin xyz="0 0 0" rpy="0 0 0"/>
       <mass value="${base_mass}"/>
@@ -35,5 +35,5 @@
         iyy="${base_mass / 12.0 * (base_height*base_height + base_width*base_width)}" iyz="0.0"
         izz="${base_mass / 12.0 * (base_width*base_width + base_length*base_length)}"/>
-      </inertial>
+      </inertial> -->
     </link>
     <joint name="left_wheel_joint" type="continuous">
@@ -60,5 +60,5 @@
         <material name="black"/>
       </visual>
-      <inertial>
+      <!-- <inertial>
         <origin xyz="0 0 0" rpy="${PI/2} 0 0"/>
         <mass value="${wheel_mass}"/>
@@ -67,5 +67,5 @@
           iyy="${wheel_mass / 12.0 * (3*wheel_radius*wheel_radius + wheel_len*wheel_len)}" iyz="0.0"
           izz="${wheel_mass / 2.0 * wheel_radius*wheel_radius}"/>
-        </inertial>
+        </inertial> -->
       </link>
     <joint name="right_wheel_joint" type="continuous">
@@ -92,5 +92,5 @@
         <material name="black"/>
       </visual>
-      <inertial>
+      <!-- <inertial>
         <origin xyz="0 0 0" rpy="${PI/2} 0 0"/>
         <mass value="${wheel_mass}"/>
@@ -99,5 +99,5 @@
           iyy="${wheel_mass / 12.0 * (3*wheel_radius*wheel_radius + wheel_len*wheel_len)}" iyz="0.0"
           izz="${wheel_mass / 2.0 * wheel_radius*wheel_radius}"/>
-        </inertial>
+        </inertial> -->
       </link>
     <joint name="caster_frontal_wheel_joint" type="fixed">
@@ -121,5 +121,5 @@
         <material name="white"/>
       </visual>
-      <inertial>
+      <!-- <inertial>
         <origin xyz="0 0 0" rpy="0 0 0"/>
         <mass value="${caster_wheel_mass}"/>
@@ -128,5 +128,5 @@
           iyy="${caster_wheel_mass * 0.4 * (caster_wheel_radius * caster_wheel_radius)}" iyz="0.0"
           izz="${caster_wheel_mass * 0.4 * (caster_wheel_radius * caster_wheel_radius)}"/>
-        </inertial>
+        </inertial> -->
       </link>
     <joint name="caster_rear_wheel_joint" type="fixed">
@@ -150,5 +150,5 @@
         <material name="white"/>
       </visual>
-      <inertial>
+      <!-- <inertial>
         <origin xyz="0 0 0" rpy="0 0 0"/>
         <mass value="${caster_wheel_mass}"/>
@@ -157,5 +157,5 @@
           iyy="${caster_wheel_mass * 0.4 * (caster_wheel_radius * caster_wheel_radius)}" iyz="0.0"
           izz="${caster_wheel_mass * 0.4 * (caster_wheel_radius * caster_wheel_radius)}"/>
-        </inertial>
+        </inertial> -->
       </link>
 </robot>
